Commit message: Doug Update

File: galil_description/urdf/galil.ros2_control.xacro (robot description, xacro)
@@ -4,6 +4,18 @@
     <ros2_control name="galil" type="system">
       <hardware>
-        <plugin>galil_driver/GalilSystemHardwareInterface</plugin>
-      </hardware>
+        <xacro:if value="$(arg use_simulation)">
+          <plugin>ign_ros2_control/IgnitionSystem</plugin>
+        </xacro:if>
+        <xacro:unless value="$(arg use_simulation)">
+          <xacro:if value="$(arg use_fake_hardware)">
+            <plugin>mock_components/GenericSystem</plugin>
+          </xacro:if>
+          <xacro:unless value="$(arg use_fake_hardware)">
+            <plugin>galil_driver/GalilSystemHardwareInterface</plugin>
+            <param name="ip_address">169.254.0.51</param>
+            <param name="check_timeout">0.1</param>
+          </xacro:unless>
+        </xacro:unless>
+     </hardware>
       <joint name="insertion_joint">
         <command_interface name="position">
@@ -16,4 +28,6 @@
         </command_interface>
         <command_interface name="real_velocity"/>
+	<param name="gear_ratio">1.0</param>
+        <param name="torque_constant">1.0</param>
         <param name="real_velocity_kp">100</param>
         <param name="real_velocity_ki">0</param>
@@ -26,4 +40,5 @@
         </state_interface>
         <state_interface name="velocity"/>
+        <state_interface name="effort"/>
       </joint>
       <joint name="horizontal_joint">
@@ -37,4 +52,6 @@
         </command_interface>
         <command_interface name="real_velocity"/>
+        <param name="gear_ratio">1.0</param>
+        <param name="torque_constant">1.0</param>
         <param name="real_velocity_kp">100</param>
         <param name="real_velocity_ki">0</param>
@@ -47,4 +64,5 @@
         </state_interface>
         <state_interface name="velocity"/>
+        <state_interface name="effort"/>
       </joint>
       <joint name="vertical_joint">
@@ -58,4 +76,6 @@
         </command_interface>
         <command_interface name="real_velocity"/>
+        <param name="gear_ratio">1.0</param>
+        <param name="torque_constant">1.0</param>
         <param name="real_velocity_kp">100</param>
         <param name="real_velocity_ki">0</param>
@@ -68,4 +88,5 @@
         </state_interface>
         <state_interface name="velocity"/>
+        <state_interface name="effort"/>
       </joint>
       <joint name="needle_drive_joint">
@@ -79,4 +100,6 @@
         </command_interface>
         <command_interface name="real_velocity"/>
+        <param name="gear_ratio">1.0</param>
+        <param name="torque_constant">1.0</param>
         <param name="real_velocity_kp">35</param>
         <param name="real_velocity_ki">0</param>
@@ -89,6 +112,13 @@
         </state_interface>
         <state_interface name="velocity"/>
+        <state_interface name="effort"/>
       </joint>
     </ros2_control>
+    <gazebo>
+      <plugin filename="libign_ros2_control-system.so" name="ign_ros2_control::IgnitionROS2ControlPlugin">
+        <parameters>$(find galil_driver)/config/galil_controllers.yaml</parameters>
+        <controller_manager_node_name>controller_manager</controller_manager_node_name>
+      </plugin>
+    </gazebo>
   </xacro:macro>
 </robot>

File: galil_description/urdf/galil.xacro (robot description, xacro)
@@ -11,4 +11,16 @@
         <material name="silver"/>
       </visual>
+      <collision>
+        <origin xyz="0 0 -0.025" rpy="0 0 ${-pi/2}"/>
+        <geometry>
+          <mesh filename="package://galil_description/meshes/base_link.stl"/>
+        </geometry>
+        <material name="silver"/>
+      </collision>
+      <inertial>
+        <mass value="1.0"/>
+        <origin xyz="0 0 0" rpy="0 0 0"/>
+        <inertia ixx="0.01" ixy="0.0" ixz="0.0" iyy="0.01" iyz="0.0" izz="0.01"/>
+      </inertial>
     </link>
     <link name="vertical_link">
@@ -20,4 +32,9 @@
         <material name="silver"/>
       </visual>
+      <inertial>
+        <mass value="1.0"/>
+        <origin xyz="0 0 0" rpy="0 0 0"/>
+        <inertia ixx="0.01" ixy="0.0" ixz="0.0" iyy="0.01" iyz="0.0" izz="0.01"/>
+      </inertial>
     </link>
     <link name="horizontal_link">
@@ -29,4 +46,9 @@
         <material name="silver"/>
       </visual>
+      <inertial>
+        <mass value="1.0"/>
+        <origin xyz="0 0 0" rpy="0 0 0"/>
+        <inertia ixx="0.01" ixy="0.0" ixz="0.0" iyy="0.01" iyz="0.0" izz="0.01"/>
+      </inertial>
     </link>
     <link name="needle_link">
@@ -38,4 +60,9 @@
         <material name="silver"/>
       </visual>
+      <inertial>
+        <mass value="1.0"/>
+        <origin xyz="0 0 0" rpy="0 0 0"/>
+        <inertia ixx="0.01" ixy="0.0" ixz="0.0" iyy="0.01" iyz="0.0" izz="0.01"/>
+      </inertial>
     </link>
     <link name="needle_drive_link">
@@ -47,4 +74,9 @@
         <material name="silver"/>
       </visual>
+      <inertial>
+        <mass value="1.0"/>
+        <origin xyz="0 0 0" rpy="0 0 0"/>
+        <inertia ixx="0.01" ixy="0.0" ixz="0.0" iyy="0.01" iyz="0.0" izz="0.01"/>
+      </inertial>
     </link>
     <joint name="vertical_joint" type="prismatic">
@@ -72,5 +104,5 @@
       <origin xyz="0 0 0" rpy="0 0 0"/>
       <parent link="horizontal_link"/>
-      <child link="needle__drive_link"/>
+      <child link="needle_drive_link"/>
       <axis xyz="0.0 1.0 0.0"/>
       <limit upper="0.1" lower="0.0" effort="100" velocity="100"/>
